File: hardware/openpod/_autosave-buttons.kicad_sch (KiCad schematic)
At the start: 8 parts

Commit message: designed clickwheel and see if mpr121 can fit on it
Parts:
- clickwheel-connector1: Manufacturer (none) -> Hirose; Part number (none) -> FH12-8S-0.5SH(55); Supplier (none) -> DigiKey; Supplier Part number (none) -> H124618TR-ND
Changed lines of the file:
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@@
       (effects (font (size 1.27 1.27)) hide)
     )
-    (property "Datasheet" "" (at 79.248 24.384 0)
+    (property "Datasheet" "https://www.mouser.fr/datasheet/2/185/FH12_8S_0_5SH_55__CL0586_0744_5_55_2DDrawing_00009-1614795.pdf" (at 79.248 24.384 0)
       (effects (font (size 1.27 1.27)) hide)
     )
-    (property "Manufacturer" "" (at 79.248 24.384 0)
+    (property "Manufacturer" "Hirose" (at 79.248 24.384 0)
       (effects (font (size 1.27 1.27)) hide)
     )
-    (property "Part number" "" (at 79.248 24.384 0)
+    (property "Part number" "FH12-8S-0.5SH(55)" (at 79.248 24.384 0)
       (effects (font (size 1.27 1.27)) hide)
     )
-    (property "Supplier" "" (at 79.248 24.384 0)
+    (property "Supplier" "DigiKey" (at 79.248 24.384 0)
       (effects (font (size 1.27 1.27)) hide)
     )
-    (property "Supplier Part number" "" (at 79.248 24.384 0)
+    (property "Supplier Part number" "H124618TR-ND" (at 79.248 24.384 0)
       (effects (font (size 1.27 1.27)) hide)
     )
