File: hardware/openpod/buttons.kicad_sch (KiCad schematic)
At the start: 6 parts

Commit message: Rebirth (#2)
* designed clickwheel and see if mpr121 can fit on it

* update power and audio

* added UART converter

* added bluetooth

* try up with vs1053 feather

* setupt the player file

* fill screen with different colors

* almost works with GFX, just wrong coordinates

* test MADCTL 1

* wrong, screen is all white

* screen pins before remap

* new pinout with consecutive 16bits on the PCs pins

* screen works

* added demo

* updated platformio.ini

* added blog

* cleanup

* first menu

* Fast (ugly) menu renderer

* ugly theme + blog post

* transition using HW scrolling

* breakdown ui

* 30 rows buffer

* remove row/col shit

* added content for the blog

* start restoring render of the now playing

* scroll to nowplaying

* working transitiontotracklist (but slight prolbem with last line)

* fixed the wrapping issue at the bottom

* update theme

* rewired vs1053

* screen and mp3 working

* pins

* updated mp3 pinout to have i2c available

* testing the clickwheel with teleplot: looking good !

* Debugging the wheel: it follows my finger on the screen

* first scrolling the tracks with the wheel !

* WIP

* use an app state and allow to use more bits per pixel

* setup unit tests

* std

* remove select track

* use doctest and reporter

* make tests pass

* cleanup

* fixed scripts

* faster render fonts

* dark background

* better state + events handler system

* wip

* faster renderer of tracklist + animations + better split between concerns

* 2 bits per pixel

* docs

* remove unit tests

* simplify ui list

* rename track to element

* rename track to element

* psram controller

* psram works on SPI1

* psram controller works

* indexer

* crawler

* radix tree?

* update trie generator

* started implementing storage

* trie index

* search works on the stm32

* can retrieve now paths

* sound player on the way

* enhanced mp3 working, but not flac

* flac plugin

* config files

* load flac plugin correctly: saccaded sound

* cleaning up

*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
Parts:
- removed MPR1: MPR121QR2, Package_DFN_QFN:UQFN-20_3x3mm_P0.4mm, symbol Sensor_Touch:MPR121QR2
- added Clickwheel1: ~, openpod:clickwheel_1, symbol openpod:clickwheel
- added MPR1: MPR121QR2, openpod:mpr121qr2, symbol openpod:MPR121QR2
- added clickwheel-connector1, clickwheel-connector2: ~, Connector_FFC-FPC:Hirose_FH12-8S-0.5SH_1x08-1MP_P0.50mm_Horizontal, symbol openpod:clickwheel-connector
Connections:
- new net: MPR1.20 (VDD), clickwheel-connector1.1 (VDD)
- new net: MPR1.1 (~{IRQ}), clickwheel-connector1.2 (IRQ)
- new net: MPR1.2 (SCL), clickwheel-connector1.3 (SCL)
- new net: MPR1.3 (SDA), clickwheel-connector1.4 (SDA)
- new net: MPR1.4 (ADDR), clickwheel-connector1.5 (ADDR)
- new net: MPR1.5 (VREG), clickwheel-connector1.6 (VREG)
- new net: MPR1.6 (VSS), clickwheel-connector1.7 (VSS)
- new net: MPR1.7 (REXT), clickwheel-connector1.8 (REXT)
- new net: Clickwheel1.1 (top), MPR1.16 (ELEC8)
- new net: Clickwheel1.2 (right), MPR1.15 (ELEC7)
- new net: Clickwheel1.3 (bottom), MPR1.19 (ELEC11)
- new net: Clickwheel1.4 (left), MPR1.9 (ELEC1)
- no-connect marks 0 -> 7
