File: hardware/openpod/openpod.kicad_sch (KiCad schematic)
At the start: 3 parts, among them U1 STM32F446RCTx

Commit message: dev boards
Other:
- added sheet BT Devboard (bt_devboard.kicad_sch)
- added sheet click-wheel-base-devboard (click-wheel-base-devboard.kicad_sch)
