File: hardware/opentone/audio.kicad_sch (KiCad schematic)
At the start: 29 parts

Commit message: Rename (#3)
* added dot when on a page with blank characters

* rename

* actions only on new version tag on master
Parts:
- Jack1: footprint openpod:CUI_SJ1-3524NG -> opentone:CUI_SJ1-3524NG; symbol openpod:SJ1-3524NG -> opentone:SJ1-3524NG
- VS1: symbol openpod:vs1063 -> opentone:vs1063
Changed lines of the file:
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@@
 		)
 		(instances
-			(project "openpod"
+			(project "opentone"
 				(path "/0122bb8c-dbef-4db1-a6c6-9be780a38d9f/624e7c04-d7d5-4e26-80cd-388aaab1d060"
 					(reference "#PWR09")
@@
 		)
 		(instances
-			(project "openpod"
+			(project "opentone"
 				(path "/0122bb8c-dbef-4db1-a6c6-9be780a38d9f/624e7c04-d7d5-4e26-80cd-388aaab1d060"
 					(reference "C34")
@@
 		)
 		(instances
-			(project "openpod"
+			(project "opentone"
 				(path "/0122bb8c-dbef-4db1-a6c6-9be780a38d9f/624e7c04-d7d5-4e26-80cd-388aaab1d060"
 					(reference "C39")
@@
 		)
 		(instances
-			(project "openpod"
+			(project "opentone"
 				(path "/0122bb8c-dbef-4db1-a6c6-9be780a38d9f/624e7c04-d7d5-4e26-80cd-388aaab1d060"
 					(reference "#PWR018")
@@
 		)
 		(instances
-			(project "openpod"
+			(project "opentone"
 				(path "/0122bb8c-dbef-4db1-a6c6-9be780a38d9f/624e7c04-d7d5-4e26-80cd-388aaab1d060"
 					(reference "C3")
@@
 		)
 		(instances
-			(project "openpod"
+			(project "opentone"
 				(path "/0122bb8c-dbef-4db1-a6c6-9be780a38d9f/624e7c04-d7d5-4e26-80cd-388aaab1d060"
 					(reference "C32")
@@
 		)
 		(instances
-			(project "openpod"
+			(project "opentone"
 				(path "/0122bb8c-dbef-4db1-a6c6-9be780a38d9f/624e7c04-d7d5-4e26-80cd-388aaab1d060"
 					(reference "#PWR014")
@@
 		)
 		(instances
-			(project "openpod"
+			(project "opentone"
 				(path "/0122bb8c-dbef-4db1-a6c6-9be780a38d9f/624e7c04-d7d5-4e26-80cd-388aaab1d060"
 					(reference "C44")
@@
 		)
 		(instances
-			(project "openpod"
+			(project "opentone"
 				(path "/0122bb8c-dbef-4db1-a6c6-9be780a38d9f/624e7c04-d7d5-4e26-80cd-388aaab1d060"
 					(reference "#PWR037")
@@
 		)
 		(instances
-			(project "openpod"
+			(project "opentone"
 				(path "/0122bb8c-dbef-4db1-a6c6-9be780a38d9f/624e7c04-d7d5-4e26-80cd-388aaab1d060"
 					(reference "R2")
@@
 		)
 		(instances
-			(project "openpod"
+			(project "opentone"
 				(path "/0122bb8c-dbef-4db1-a6c6-9be780a38d9f/624e7c04-d7d5-4e26-80cd-388aaab1d060"
 					(reference "C36")
@@
 		)
 		(instances
-			(project "openpod"
+			(project "opentone"
 				(path "/0122bb8c-dbef-4db1-a6c6-9be780a38d9f/624e7c04-d7d5-4e26-80cd-388aaab1d060"
 					(reference "#PWR017")
@@
 		)
 		(instances
-			(project "openpod"
+			(project "opentone"
 				(path "/0122bb8c-dbef-4db1-a6c6-9be780a38d9f/624e7c04-d7d5-4e26-80cd-388aaab1d060"
 					(reference "#PWR015")
@@
 		)
 		(instances
-			(project "openpod"
+			(project "opentone"
 				(path "/0122bb8c-dbef-4db1-a6c6-9be780a38d9f/624e7c04-d7d5-4e26-80cd-388aaab1d060"
 					(reference "#PWR027")
@@
 		)
 		(instances
-			(project "openpod"
+			(project "opentone"
 				(path "/0122bb8c-dbef-4db1-a6c6-9be780a38d9f/624e7c04-d7d5-4e26-80cd-388aaab1d060"
 					(reference "C35")
@@
 		)
 		(instances
-			(project "openpod"
+			(project "opentone"
 				(path "/0122bb8c-dbef-4db1-a6c6-9be780a38d9f/624e7c04-d7d5-4e26-80cd-388aaab1d060"
 					(reference "C45")
@@
 		)
 		(instances
-			(project "openpod"
+			(project "opentone"
 				(path "/0122bb8c-dbef-4db1-a6c6-9be780a38d9f/624e7c04-d7d5-4e26-80cd-388aaab1d060"
 					(reference "#PWR013")
@@
 		)
 		(instances
-			(project "openpod"
+			(project "opentone"
 				(path "/0122bb8c-dbef-4db1-a6c6-9be780a38d9f/624e7c04-d7d5-4e26-80cd-388aaab1d060"
 					(reference "#PWR033")
@@
 		)
 		(instances
-			(project "openpod"
+			(project "opentone"
 				(path "/0122bb8c-dbef-4db1-a6c6-9be780a38d9f/624e7c04-d7d5-4e26-80cd-388aaab1d060"
 					(reference "Cristal1")
@@
 		)
 		(instances
-			(project "openpod"
+			(project "opentone"
 				(path "/0122bb8c-dbef-4db1-a6c6-9be780a38d9f/624e7c04-d7d5-4e26-80cd-388aaab1d060"
 					(reference "C40")
@@
 		)
 		(instances
-			(project "openpod"
+			(project "opentone"
 				(path "/0122bb8c-dbef-4db1-a6c6-9be780a38d9f/624e7c04-d7d5-4e26-80cd-388aaab1d060"
 					(reference "R18")
@@
 		)
 		(instances
-			(project "openpod"
+			(project "opentone"
 				(path "/0122bb8c-dbef-4db1-a6c6-9be780a38d9f/624e7c04-d7d5-4e26-80cd-388aaab1d060"
 					(reference "R13")
@@
 		)
 		(instances
-			(project "openpod"
+			(project "opentone"
 				(path "/0122bb8c-dbef-4db1-a6c6-9be780a38d9f/624e7c04-d7d5-4e26-80cd-388aaab1d060"
 					(reference "C42")
@@
 		)
 		(instances
-			(project "openpod"
+			(project "opentone"
 				(path "/0122bb8c-dbef-4db1-a6c6-9be780a38d9f/624e7c04-d7d5-4e26-80cd-388aaab1d060"
 					(reference "C33")
@@
 		)
 		(instances
-			(project "openpod"
+			(project "opentone"
 				(path "/0122bb8c-dbef-4db1-a6c6-9be780a38d9f/624e7c04-d7d5-4e26-80cd-388aaab1d060"
 					(reference "C29")
@@
 		)
 		(instances
-			(project "openpod"
+			(project "opentone"
 				(path "/0122bb8c-dbef-4db1-a6c6-9be780a38d9f/624e7c04-d7d5-4e26-80cd-388aaab1d060"
 					(reference "R14")
@@
 		)
 		(instances
-			(project "openpod"
+			(project "opentone"
 				(path "/0122bb8c-dbef-4db1-a6c6-9be780a38d9f/624e7c04-d7d5-4e26-80cd-388aaab1d060"
 					(reference "#PWR08")
@@
 		)
 		(instances
-			(project "openpod"
+			(project "opentone"
 				(path "/0122bb8c-dbef-4db1-a6c6-9be780a38d9f/624e7c04-d7d5-4e26-80cd-388aaab1d060"
 					(reference "C30")
@@
 		)
 		(instances
-			(project "openpod"
+			(project "opentone"
 				(path "/0122bb8c-dbef-4db1-a6c6-9be780a38d9f/624e7c04-d7d5-4e26-80cd-388aaab1d060"
 					(reference "#PWR038")
@@
 		)
 		(instances
-			(project "openpod"
+			(project "opentone"
 				(path "/0122bb8c-dbef-4db1-a6c6-9be780a38d9f/624e7c04-d7d5-4e26-80cd-388aaab1d060"
 					(reference "C9")
@@
 	)
 	(symbol
-		(lib_id "openpod:SJ1-3524NG")
+		(lib_id "opentone:SJ1-3524NG")
 		(at 74.676 69.596 270)
 		(unit 1)
@@
 			)
 		)
-		(property "Footprint" "openpod:CUI_SJ1-3524NG"
+		(property "Footprint" "opentone:CUI_SJ1-3524NG"
 			(at 74.676 69.596 0)
 			(effects
@@
 		)
 		(instances
-			(project "openpod"
+			(project "opentone"
 				(path "/0122bb8c-dbef-4db1-a6c6-9be780a38d9f/624e7c04-d7d5-4e26-80cd-388aaab1d060"
 					(reference "Jack1")
@@
 		)
 		(instances
-			(project "openpod"
+			(project "opentone"
 				(path "/0122bb8c-dbef-4db1-a6c6-9be780a38d9f/624e7c04-d7d5-4e26-80cd-388aaab1d060"
 					(reference "C31")
@@
 		)
 		(instances
-			(project "openpod"
+			(project "opentone"
 				(path "/0122bb8c-dbef-4db1-a6c6-9be780a38d9f/624e7c04-d7d5-4e26-80cd-388aaab1d060"
 					(reference "C43")
@@
 		)
 		(instances
-			(project "openpod"
+			(project "opentone"
 				(path "/0122bb8c-dbef-4db1-a6c6-9be780a38d9f/624e7c04-d7d5-4e26-80cd-388aaab1d060"
 					(reference "R17")
@@
 		)
 		(instances
-			(project "openpod"
+			(project "opentone"
 				(path "/0122bb8c-dbef-4db1-a6c6-9be780a38d9f/624e7c04-d7d5-4e26-80cd-388aaab1d060"
 					(reference "R16")
@@
 		)
 		(instances
-			(project "openpod"
+			(project "opentone"
 				(path "/0122bb8c-dbef-4db1-a6c6-9be780a38d9f/624e7c04-d7d5-4e26-80cd-388aaab1d060"
 					(reference "#PWR016")
@@
 		)
 		(instances
-			(project "openpod"
+			(project "opentone"
 				(path "/0122bb8c-dbef-4db1-a6c6-9be780a38d9f/624e7c04-d7d5-4e26-80cd-388aaab1d060"
 					(reference "#PWR012")
@@
 		)
 		(instances
-			(project "openpod"
+			(project "opentone"
 				(path "/0122bb8c-dbef-4db1-a6c6-9be780a38d9f/624e7c04-d7d5-4e26-80cd-388aaab1d060"
 					(reference "C37")
@@
 		)
 		(instances
-			(project "openpod"
+			(project "opentone"
 				(path "/0122bb8c-dbef-4db1-a6c6-9be780a38d9f/624e7c04-d7d5-4e26-80cd-388aaab1d060"
 					(reference "C38")
@@
 		)
 		(instances
-			(project "openpod"
+			(project "opentone"
 				(path "/0122bb8c-dbef-4db1-a6c6-9be780a38d9f/624e7c04-d7d5-4e26-80cd-388aaab1d060"
 					(reference "C41")
@@
 	)
 	(symbol
-		(lib_id "openpod:vs1063")
+		(lib_id "opentone:vs1063")
 		(at 158.242 66.04 0)
 		(unit 1)
@@
 		)
 		(instances
-			(project "openpod"
+			(project "opentone"
 				(path "/0122bb8c-dbef-4db1-a6c6-9be780a38d9f/624e7c04-d7d5-4e26-80cd-388aaab1d060"
 					(reference "VS1")
@@
 		)
 		(instances
-			(project "openpod"
+			(project "opentone"
 				(path "/0122bb8c-dbef-4db1-a6c6-9be780a38d9f/624e7c04-d7d5-4e26-80cd-388aaab1d060"
 					(reference "R3")
