File: hardware/opentone/bt_devboard.kicad_pcb (KiCad board)
At the start: 2 copper layers, 52 x 46 mm, 7 parts, among them J101 POWER, J2 Conn_01x09, SW101 PWR, SW102 RST, U101 FSC-BT1035

Commit message: Rename (#3)
* added dot when on a page with blank characters

* rename

* actions only on new version tag on master
Parts:
- U101: footprint openpod:fsc-bt1035 -> opentone:fsc-bt1035
Changed lines of the file:
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@@
 		)
 	)
-	(footprint "openpod:fsc-bt1035"
+	(footprint "opentone:fsc-bt1035"
 		(layer "F.Cu")
 		(at 105.315 59 180)
