File: hardware/opentone/click-wheel-base-devboard.kicad_pcb (KiCad board)
At the start: 2 copper layers, 36 x 50 mm, 11 parts, among them J2 Conn_01x09

Commit message: Rename (#3)
* added dot when on a page with blank characters

* rename

* actions only on new version tag on master
Parts:
- cwdev-bottom, cwdev-center, cwdev-left, cwdev-right, cwdev-top: footprint openpod:SW_SKQGAFE010 -> opentone:SW_SKQGAFE010
Changed lines of the file:
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@@
 		)
 	)
-	(footprint "openpod:SW_SKQGAFE010"
+	(footprint "opentone:SW_SKQGAFE010"
 		(layer "F.Cu")
 		(at 89 79)
@@
 		)
 	)
-	(footprint "openpod:SW_SKQGAFE010"
+	(footprint "opentone:SW_SKQGAFE010"
 		(layer "F.Cu")
 		(at 101 67)
@@
 		)
 	)
-	(footprint "openpod:SW_SKQGAFE010"
+	(footprint "opentone:SW_SKQGAFE010"
 		(layer "F.Cu")
 		(at 77 67)
@@
 		)
 	)
-	(footprint "openpod:SW_SKQGAFE010"
+	(footprint "opentone:SW_SKQGAFE010"
 		(layer "F.Cu")
 		(at 89 55)
@@
 		)
 	)
-	(footprint "openpod:SW_SKQGAFE010"
+	(footprint "opentone:SW_SKQGAFE010"
 		(layer "F.Cu")
 		(at 89 67)
