File: hardware/opentone/opentone.kicad_pcb (KiCad board)
At the start: 2 copper layers, 161.1 x 143.3 mm, 35 parts, among them J101 POWER, J102 UART, J103 DEBUG, J104 USB, SW101 PWR, SW102 RST, U1 STM32F446RCTx, U101 FSC-BT1035

Commit message: Rename (#3)
* added dot when on a page with blank characters

* rename

* actions only on new version tag on master
Parts:
- removed Bluetooth: ~, openpod:fsc-bt1035
- removed FSC_BT-1: ~, openpod:fsc-bt1046
- Clickwheel1: footprint openpod:clickwheel_1 -> opentone:clickwheel_1
- Jack1: footprint openpod:CUI_SJ1-3524NG -> opentone:CUI_SJ1-3524NG
- MPR1: footprint openpod:mpr121qr2 -> opentone:mpr121qr2
- SCREEN1: footprint openpod:nhd-2.4-240320cf-ctxif -> opentone:nhd-2.4-240320cf-ctxif
- S_CONNECTOR1: footprint openpod:Hirose_FH12-40S-0.5SH_1x40-1MP_P0.50mm_Horizontal -> opentone:Hirose_FH12-40S-0.5SH_1x40-1MP_P0.50mm_Horizontal
- U101: footprint openpod:fsc-bt1035 -> opentone:fsc-bt1035
- bottom1, center1, left1, right1, top1: footprint openpod:SW_SKQGAFE010 -> opentone:SW_SKQGAFE010
- moved U101 61.1 mm to (27.5, 111.0)
Routing:
- added copper zone on B.Cu, net GND
