File: hardware/opentone/opentone.kicad_sch (KiCad schematic)
At the start: 3 parts, among them U1 STM32F446RCTx

Commit message: Rename (#3)
* added dot when on a page with blank characters

* rename

* actions only on new version tag on master
Parts:
- SCREEN1: footprint openpod:nhd-2.4-240320cf-ctxif -> opentone:nhd-2.4-240320cf-ctxif
- S_CONNECTOR1: footprint openpod:Hirose_FH12-40S-0.5SH_1x40-1MP_P0.50mm_Horizontal -> opentone:Hirose_FH12-40S-0.5SH_1x40-1MP_P0.50mm_Horizontal
Changed lines of the file:
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@@
 		)
 		(instances
-			(project "openpod"
+			(project "opentone"
 				(path "/0122bb8c-dbef-4db1-a6c6-9be780a38d9f"
 					(reference "U1")
@@
 			)
 		)
-		(property "Footprint" "openpod:nhd-2.4-240320cf-ctxif"
+		(property "Footprint" "opentone:nhd-2.4-240320cf-ctxif"
 			(at 259.08 35.56 0)
 			(effects
@@
 		)
 		(instances
-			(project "openpod"
+			(project "opentone"
 				(path "/0122bb8c-dbef-4db1-a6c6-9be780a38d9f"
 					(reference "SCREEN1")
@@
 			)
 		)
-		(property "Footprint" "openpod:Hirose_FH12-40S-0.5SH_1x40-1MP_P0.50mm_Horizontal"
+		(property "Footprint" "opentone:Hirose_FH12-40S-0.5SH_1x40-1MP_P0.50mm_Horizontal"
 			(at 203.2 35.56 0)
 			(effects
@@
 		)
 		(instances
-			(project "openpod"
+			(project "opentone"
 				(path "/0122bb8c-dbef-4db1-a6c6-9be780a38d9f"
 					(reference "S_CONNECTOR1")
@@
 		)
 		(instances
-			(project "openpod"
+			(project "opentone"
 				(path "/0122bb8c-dbef-4db1-a6c6-9be780a38d9f"
 					(page "3")
@@
 		)
 		(instances
-			(project "openpod"
+			(project "opentone"
 				(path "/0122bb8c-dbef-4db1-a6c6-9be780a38d9f"
 					(page "4")
@@
 		)
 		(instances
-			(project "openpod"
+			(project "opentone"
 				(path "/0122bb8c-dbef-4db1-a6c6-9be780a38d9f"
 					(page "7")
@@
 		)
 		(instances
-			(project "openpod"
+			(project "opentone"
 				(path "/0122bb8c-dbef-4db1-a6c6-9be780a38d9f"
 					(page "5")
@@
 		)
 		(instances
-			(project "openpod"
+			(project "opentone"
 				(path "/0122bb8c-dbef-4db1-a6c6-9be780a38d9f"
 					(page "2")
