File: hardware/opentone/power.kicad_sch (KiCad schematic)
At the start: 32 parts

Commit message: Rename (#3)
* added dot when on a page with blank characters

* rename

* actions only on new version tag on master
Parts:
- AP7312: symbol openpod:AP7312 -> opentone:AP7312
Changed lines of the file:
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@@
 		)
 		(instances
-			(project "openpod"
+			(project "opentone"
 				(path "/0122bb8c-dbef-4db1-a6c6-9be780a38d9f/ddcf786c-06d2-421e-b65a-77775151c20a"
 					(reference "D4")
@@
 		)
 		(instances
-			(project "openpod"
+			(project "opentone"
 				(path "/0122bb8c-dbef-4db1-a6c6-9be780a38d9f/ddcf786c-06d2-421e-b65a-77775151c20a"
 					(reference "D6")
@@
 		)
 		(instances
-			(project "openpod"
+			(project "opentone"
 				(path "/0122bb8c-dbef-4db1-a6c6-9be780a38d9f/ddcf786c-06d2-421e-b65a-77775151c20a"
 					(reference "C48")
@@
 		)
 		(instances
-			(project "openpod"
+			(project "opentone"
 				(path "/0122bb8c-dbef-4db1-a6c6-9be780a38d9f/ddcf786c-06d2-421e-b65a-77775151c20a"
 					(reference "C2")
@@
 		)
 		(instances
-			(project "openpod"
+			(project "opentone"
 				(path "/0122bb8c-dbef-4db1-a6c6-9be780a38d9f/ddcf786c-06d2-421e-b65a-77775151c20a"
 					(reference "#PWR041")
@@
 		)
 		(instances
-			(project "openpod"
+			(project "opentone"
 				(path "/0122bb8c-dbef-4db1-a6c6-9be780a38d9f/ddcf786c-06d2-421e-b65a-77775151c20a"
 					(reference "C49")
@@
 		)
 		(instances
-			(project "openpod"
+			(project "opentone"
 				(path "/0122bb8c-dbef-4db1-a6c6-9be780a38d9f/ddcf786c-06d2-421e-b65a-77775151c20a"
 					(reference "F2")
@@
 		)
 		(instances
-			(project "openpod"
+			(project "opentone"
 				(path "/0122bb8c-dbef-4db1-a6c6-9be780a38d9f/ddcf786c-06d2-421e-b65a-77775151c20a"
 					(reference "#PWR04")
@@
 		)
 		(instances
-			(project "openpod"
+			(project "opentone"
 				(path "/0122bb8c-dbef-4db1-a6c6-9be780a38d9f/ddcf786c-06d2-421e-b65a-77775151c20a"
 					(reference "#PWR010")
@@
 		)
 		(instances
-			(project "openpod"
+			(project "opentone"
 				(path "/0122bb8c-dbef-4db1-a6c6-9be780a38d9f/ddcf786c-06d2-421e-b65a-77775151c20a"
 					(reference "#PWR011")
@@
 		)
 		(instances
-			(project "openpod"
+			(project "opentone"
 				(path "/0122bb8c-dbef-4db1-a6c6-9be780a38d9f/ddcf786c-06d2-421e-b65a-77775151c20a"
 					(reference "UART_BRIDGE1")
@@
 		)
 		(instances
-			(project "openpod"
+			(project "opentone"
 				(path "/0122bb8c-dbef-4db1-a6c6-9be780a38d9f/ddcf786c-06d2-421e-b65a-77775151c20a"
 					(reference "#PWR042")
@@
 		)
 		(instances
-			(project "openpod"
+			(project "opentone"
 				(path "/0122bb8c-dbef-4db1-a6c6-9be780a38d9f/ddcf786c-06d2-421e-b65a-77775151c20a"
 					(reference "D5")
@@
 		)
 		(instances
-			(project "openpod"
+			(project "opentone"
 				(path "/0122bb8c-dbef-4db1-a6c6-9be780a38d9f/ddcf786c-06d2-421e-b65a-77775151c20a"
 					(reference "R5")
@@
 		)
 		(instances
-			(project "openpod"
+			(project "opentone"
 				(path "/0122bb8c-dbef-4db1-a6c6-9be780a38d9f/ddcf786c-06d2-421e-b65a-77775151c20a"
 					(reference "C1")
@@
 		)
 		(instances
-			(project "openpod"
+			(project "opentone"
 				(path "/0122bb8c-dbef-4db1-a6c6-9be780a38d9f/ddcf786c-06d2-421e-b65a-77775151c20a"
 					(reference "FB1")
@@
 		)
 		(instances
-			(project "openpod"
+			(project "opentone"
 				(path "/0122bb8c-dbef-4db1-a6c6-9be780a38d9f/ddcf786c-06d2-421e-b65a-77775151c20a"
 					(reference "#PWR03")
@@
 		)
 		(instances
-			(project "openpod"
+			(project "opentone"
 				(path "/0122bb8c-dbef-4db1-a6c6-9be780a38d9f/ddcf786c-06d2-421e-b65a-77775151c20a"
 					(reference "C46")
@@
 		)
 		(instances
-			(project "openpod"
+			(project "opentone"
 				(path "/0122bb8c-dbef-4db1-a6c6-9be780a38d9f/ddcf786c-06d2-421e-b65a-77775151c20a"
 					(reference "USB1")
@@
 		)
 		(instances
-			(project "openpod"
+			(project "opentone"
 				(path "/0122bb8c-dbef-4db1-a6c6-9be780a38d9f/ddcf786c-06d2-421e-b65a-77775151c20a"
 					(reference "R1")
@@
 		)
 		(instances
-			(project "openpod"
+			(project "opentone"
 				(path "/0122bb8c-dbef-4db1-a6c6-9be780a38d9f/ddcf786c-06d2-421e-b65a-77775151c20a"
 					(reference "R6")
@@
 		)
 		(instances
-			(project "openpod"
+			(project "opentone"
 				(path "/0122bb8c-dbef-4db1-a6c6-9be780a38d9f/ddcf786c-06d2-421e-b65a-77775151c20a"
 					(reference "#PWR05")
@@
 		)
 		(instances
-			(project "openpod"
+			(project "opentone"
 				(path "/0122bb8c-dbef-4db1-a6c6-9be780a38d9f/ddcf786c-06d2-421e-b65a-77775151c20a"
 					(reference "C4")
@@
 		)
 		(instances
-			(project "openpod"
+			(project "opentone"
 				(path "/0122bb8c-dbef-4db1-a6c6-9be780a38d9f/ddcf786c-06d2-421e-b65a-77775151c20a"
 					(reference "#PWR06")
@@
 		)
 		(instances
-			(project "openpod"
+			(project "opentone"
 				(path "/0122bb8c-dbef-4db1-a6c6-9be780a38d9f/ddcf786c-06d2-421e-b65a-77775151c20a"
 					(reference "#PWR01")
@@
 		)
 		(instances
-			(project "openpod"
+			(project "opentone"
 				(path "/0122bb8c-dbef-4db1-a6c6-9be780a38d9f/ddcf786c-06d2-421e-b65a-77775151c20a"
 					(reference "#PWR019")
@@
 		)
 		(instances
-			(project "openpod"
+			(project "opentone"
 				(path "/0122bb8c-dbef-4db1-a6c6-9be780a38d9f/ddcf786c-06d2-421e-b65a-77775151c20a"
 					(reference "R19")
@@
 		)
 		(instances
-			(project "openpod"
+			(project "opentone"
 				(path "/0122bb8c-dbef-4db1-a6c6-9be780a38d9f/ddcf786c-06d2-421e-b65a-77775151c20a"
 					(reference "#PWR020")
@@
 		)
 		(instances
-			(project "openpod"
+			(project "opentone"
 				(path "/0122bb8c-dbef-4db1-a6c6-9be780a38d9f/ddcf786c-06d2-421e-b65a-77775151c20a"
 					(reference "C52")
@@
 		)
 		(instances
-			(project "openpod"
+			(project "opentone"
 				(path "/0122bb8c-dbef-4db1-a6c6-9be780a38d9f/ddcf786c-06d2-421e-b65a-77775151c20a"
 					(reference "R7")
@@
 		)
 		(instances
-			(project "openpod"
+			(project "opentone"
 				(path "/0122bb8c-dbef-4db1-a6c6-9be780a38d9f/ddcf786c-06d2-421e-b65a-77775151c20a"
 					(reference "C50")
@@
 		)
 		(instances
-			(project "openpod"
+			(project "opentone"
 				(path "/0122bb8c-dbef-4db1-a6c6-9be780a38d9f/ddcf786c-06d2-421e-b65a-77775151c20a"
 					(reference "L2")
@@
 		)
 		(instances
-			(project "openpod"
+			(project "opentone"
 				(path "/0122bb8c-dbef-4db1-a6c6-9be780a38d9f/ddcf786c-06d2-421e-b65a-77775151c20a"
 					(reference "#PWR039")
@@
 		)
 		(instances
-			(project "openpod"
+			(project "opentone"
 				(path "/0122bb8c-dbef-4db1-a6c6-9be780a38d9f/ddcf786c-06d2-421e-b65a-77775151c20a"
 					(reference "R4")
@@
 		)
 		(instances
-			(project "openpod"
+			(project "opentone"
 				(path "/0122bb8c-dbef-4db1-a6c6-9be780a38d9f/ddcf786c-06d2-421e-b65a-77775151c20a"
 					(reference "#PWR023")
@@
 		)
 		(instances
-			(project "openpod"
+			(project "opentone"
 				(path "/0122bb8c-dbef-4db1-a6c6-9be780a38d9f/ddcf786c-06d2-421e-b65a-77775151c20a"
 					(reference "#PWR045")
@@
 		)
 		(instances
-			(project "openpod"
+			(project "opentone"
 				(path "/0122bb8c-dbef-4db1-a6c6-9be780a38d9f/ddcf786c-06d2-421e-b65a-77775151c20a"
 					(reference "FB2")
@@
 		)
 		(instances
-			(project "openpod"
+			(project "opentone"
 				(path "/0122bb8c-dbef-4db1-a6c6-9be780a38d9f/ddcf786c-06d2-421e-b65a-77775151c20a"
 					(reference "C5")
@@
 		)
 		(instances
-			(project "openpod"
+			(project "opentone"
 				(path "/0122bb8c-dbef-4db1-a6c6-9be780a38d9f/ddcf786c-06d2-421e-b65a-77775151c20a"
 					(reference "#PWR043")
@@
 		)
 		(instances
-			(project "openpod"
+			(project "opentone"
 				(path "/0122bb8c-dbef-4db1-a6c6-9be780a38d9f/ddcf786c-06d2-421e-b65a-77775151c20a"
 					(reference "#PWR044")
@@
 		)
 		(instances
-			(project "openpod"
+			(project "opentone"
 				(path "/0122bb8c-dbef-4db1-a6c6-9be780a38d9f/ddcf786c-06d2-421e-b65a-77775151c20a"
 					(reference "#PWR021")
@@
 		)
 		(instances
-			(project "openpod"
+			(project "opentone"
 				(path "/0122bb8c-dbef-4db1-a6c6-9be780a38d9f/ddcf786c-06d2-421e-b65a-77775151c20a"
 					(reference "Buck-converter2")
@@
 		)
 		(instances
-			(project "openpod"
+			(project "opentone"
 				(path "/0122bb8c-dbef-4db1-a6c6-9be780a38d9f/ddcf786c-06d2-421e-b65a-77775151c20a"
 					(reference "R21")
@@
 		)
 		(instances
-			(project "openpod"
+			(project "opentone"
 				(path "/0122bb8c-dbef-4db1-a6c6-9be780a38d9f/ddcf786c-06d2-421e-b65a-77775151c20a"
 					(reference "#PWR022")
@@
 		)
 		(instances
-			(project "openpod"
+			(project "opentone"
 				(path "/0122bb8c-dbef-4db1-a6c6-9be780a38d9f/ddcf786c-06d2-421e-b65a-77775151c20a"
 					(reference "bat-man1")
@@
 		)
 		(instances
-			(project "openpod"
+			(project "opentone"
 				(path "/0122bb8c-dbef-4db1-a6c6-9be780a38d9f/ddcf786c-06d2-421e-b65a-77775151c20a"
 					(reference "R22")
@@
 		)
 		(instances
-			(project "openpod"
+			(project "opentone"
 				(path "/0122bb8c-dbef-4db1-a6c6-9be780a38d9f/ddcf786c-06d2-421e-b65a-77775151c20a"
 					(reference "C47")
@@
 		)
 		(instances
-			(project "openpod"
+			(project "opentone"
 				(path "/0122bb8c-dbef-4db1-a6c6-9be780a38d9f/ddcf786c-06d2-421e-b65a-77775151c20a"
 					(reference "#PWR040")
@@
 		)
 		(instances
-			(project "openpod"
+			(project "opentone"
 				(path "/0122bb8c-dbef-4db1-a6c6-9be780a38d9f/ddcf786c-06d2-421e-b65a-77775151c20a"
 					(reference "#PWR02")
@@
 		)
 		(instances
-			(project "openpod"
+			(project "opentone"
 				(path "/0122bb8c-dbef-4db1-a6c6-9be780a38d9f/ddcf786c-06d2-421e-b65a-77775151c20a"
 					(reference "#PWR024")
@@
 		)
 		(instances
-			(project "openpod"
+			(project "opentone"
 				(path "/0122bb8c-dbef-4db1-a6c6-9be780a38d9f/ddcf786c-06d2-421e-b65a-77775151c20a"
 					(reference "R20")
@@
 		)
 		(instances
-			(project "openpod"
+			(project "opentone"
 				(path "/0122bb8c-dbef-4db1-a6c6-9be780a38d9f/ddcf786c-06d2-421e-b65a-77775151c20a"
 					(reference "#PWR07")
@@
 	)
 	(symbol
-		(lib_id "openpod:AP7312")
+		(lib_id "opentone:AP7312")
 		(at 200.66 70.104 0)
 		(unit 1)
@@
 		)
 		(instances
-			(project "openpod"
+			(project "opentone"
 				(path "/0122bb8c-dbef-4db1-a6c6-9be780a38d9f/ddcf786c-06d2-421e-b65a-77775151c20a"
 					(reference "AP7312")
@@
 		)
 		(instances
-			(project "openpod"
+			(project "opentone"
 				(path "/0122bb8c-dbef-4db1-a6c6-9be780a38d9f/ddcf786c-06d2-421e-b65a-77775151c20a"
 					(reference "BT2")
